File: board/TOFE-HDMI4.kicad_pcb (KiCad board)
At the start: 2 copper layers, 1 part

Commit message: Creating TOFE-HDMI4!
Parts:
- U?: value TOFE_Expansion_Board_8x_HalfHeight -> TOFE_HDMI4_Expansion_Board_8x_HalfHeight
Changed lines of the file:
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@@
       (effects (font (size 1.016 1.016) (thickness 0.254)))
     )
-    (fp_text value TOFE_Expansion_Board_8x_HalfHeight (at 27.3685 -11.3665) (layer F.SilkS) hide
+    (fp_text value TOFE_HDMI4_Expansion_Board_8x_HalfHeight (at 27.3685 -11.3665) (layer F.SilkS) hide
       (effects (font (size 1.016 1.016) (thickness 0.254)))
     )
