File: board/HDMI.sch (KiCad schematic (older format))
At the start: 91 parts, among them J2 HDMI, J3 HDMI, J4 HDMI, J5 HDMI, P10 CONN_1, P19 CONN_1, P2 CONN_1, P20 CONN_1, P21 CONN_1, P22 CONN_1, P23 CONN_1, P24 CONN_1, P25 CONN_1, P26 CONN_1, P4 CONN_1, P5 CONN_1, P6 CONN_1, P7 CONN_1, P8 CONN_1, P9 CONN_1, U13 IP4776CZ38, U14 IP4776CZ38, U15 IP4776CZ38, U16 ΜA78L00, U21 IP4776CZ38, U22 ΜA78L00, U30 ΜA78L00

Commit message: Starting to modify the schematic.
Parts:
- removed C173, C177: 0.33mfd, SM0603, symbol C
- removed C175, C181, C205, C252: 0.1mfd, SM0603, symbol C
- removed R195, R202: 100K, SM0603, symbol R
- removed U16, U22: ΜA78L00, μA78L00, symbol ΜA78L00
- renumbered P10 to H10, P19 to H19, P2 to H3, P4 to H4, J4 to J1, J5 to J2, J2 to J4
Connections:
- net labels added: H1-CEC, H1-CLK+, H1-CLK-, H1-D0+, H1-D0-, H1-D1+, H1-D1-, H1-D2+, H1-D2-, H1-HOT, H1-SCL, H1-SDA, H2-CEC, H2-CLK+, H2-CLK-, H2-D0+, H2-D0-, H2-D1+, H2-D1-, H2-D2+, H2-D2-, H2-HOT, H2-SCL, H2-SDA, H3-CEC, H3-CLK+, H3-CLK-, H3-D0+, H3-D0-, H3-D1+, H3-D1-, H3-D2+, H3-D2-, H3-HOT, H3-SCL, H3-SDA, H4-CEC, H4-CLK+, H4-CLK-, H4-D0+, H4-D0-, H4-D1+, H4-D1-, H4-D2+, H4-D2-, H4-HOT, H4-SCL, H4-SDA
- net labels removed: P1-CEC, P1-CLK+, P1-CLK-, P1-D0+, P1-D0-, P1-D1+, P1-D1-, P1-D2+, P1-D2-, P1-HOT, P1-SCL, P1-SDA, P2-CEC, P2-CLK+, P2-CLK-, P2-D0+, P2-D0-, P2-D1+, P2-D1-, P2-D2+, P2-D2-, P2-HOT, P2-SCL, P2-SDA, P3-CEC, P3-CLK+, P3-CLK-, P3-D0+, P3-D0-, P3-D1+, P3-D1-, P3-D2+, P3-D2-, P3-HOT, P3-SCL, P3-SDA, P4-CEC, P4-CLK+, P4-CLK-, P4-D0+, P4-D0-, P4-D1+, P4-D1-, P4-D2+, P4-D2-, P4-HOT, P4-SCL, P4-SDA
- wire segments 417 -> 391
Other:
- note added: "HDMI 1"
- note added: "HDMI 2"
- note added: "HDMI 3"
- note added: "HDMI 4"
- note added: "HDMI H1"
- note added: "HDMI H2"
- note added: "HDMI H3"
- note added: "HDMI H4"
- note removed: "HDMI IN 1"
- note removed: "HDMI IN 2"
- note removed: "HDMI OUT 1"
- note removed: "HDMI OUT 2"
- note removed: "HDMI P1"
- note removed: "HDMI P2"
- note removed: "HDMI P3"
- note removed: "HDMI P4"
- note removed: "LDO OUT FOR"
