File: board/HDMI.sch (KiCad schematic (older format))
At the start: 81 parts, among them J1 HDMI, J2 HDMI, J3 HDMI, J4 HDMI, P20 CONN_1, P21 CONN_1, P22 CONN_1, P23 CONN_1, P24 CONN_1, P25 CONN_1, P26 CONN_1, P5 CONN_1, P6 CONN_1, P7 CONN_1, P8 CONN_1, P9 CONN_1, U13 IP4776CZ38, U14 IP4776CZ38, U15 IP4776CZ38, U21 IP4776CZ38, U30 ΜA78L00

Commit message: More modification to the schematic.
Parts:
- removed C172, C185: 0.1mfd, SM0402, symbol C
- removed R128, R131: 50R, SM0402, symbol R
- removed R153, R205: 1K, SM0402, symbol R
- removed R84, R88: 100K, SM0603, symbol R
- added R? (x2): 50R, SM0402, symbol R
- renumbered H19 to P01, P8 to P02, P7 to P03, P24 to P04, P25 to P11, H10 to P12, P9 to P13, P26 to P14, P20 to P31, P6 to P32, P5 to P33, P21 to P34, P22 to P41, H4 to P42, H3 to P43, P23 to P44, U15 to U1, U21 to U2, U13 to U3, U14 to U4
Connections:
- net labels added: TMDS_P1_0_N, TMDS_P1_0_P, TMDS_P1_1_N, TMDS_P1_1_P, TMDS_P1_2_N, TMDS_P1_2_P, TMDS_P1_CEC, TMDS_P1_CLK_N, TMDS_P1_CLK_P, TMDS_P1_HOT, TMDS_P1_SCL, TMDS_P1_SDA, TMDS_P2_0_N, TMDS_P2_0_P, TMDS_P2_1_N, TMDS_P2_1_P, TMDS_P2_2_N, TMDS_P2_2_P, TMDS_P2_CEC, TMDS_P2_CLK_N, TMDS_P2_CLK_P, TMDS_P2_HOT, TMDS_P2_SCL, TMDS_P2_SDA, TMDS_P3_0_N, TMDS_P3_0_P, TMDS_P3_1_N, TMDS_P3_1_P, TMDS_P3_2_N, TMDS_P3_2_P, TMDS_P3_CEC, TMDS_P3_CLK_N, TMDS_P3_CLK_P, TMDS_P3_HOT, TMDS_P3_SCL, TMDS_P3_SDA, TMDS_P4_0_N, TMDS_P4_0_P, TMDS_P4_1_N, TMDS_P4_1_P, TMDS_P4_2_N, TMDS_P4_2_P, TMDS_P4_CEC, TMDS_P4_CLK_N, TMDS_P4_CLK_P, TMDS_P4_HOT, TMDS_P4_SCL, TMDS_P4_SDA, VCC5V
- net labels removed: HDMI-TX1-VCC5V0, HDMI-TX2-VCC5V0, TMDS_RX1_0_N, TMDS_RX1_0_P, TMDS_RX1_1_N, TMDS_RX1_1_P, TMDS_RX1_2_N, TMDS_RX1_2_P, TMDS_RX1_CEC, TMDS_RX1_CLK_N, TMDS_RX1_CLK_P, TMDS_RX1_HOT, TMDS_RX1_SCL, TMDS_RX1_SDA, TMDS_RX2_0_N, TMDS_RX2_0_P, TMDS_RX2_1_N, TMDS_RX2_1_P, TMDS_RX2_2_N, TMDS_RX2_2_P, TMDS_RX2_CEC, TMDS_RX2_CLK_N, TMDS_RX2_CLK_P, TMDS_RX2_HOT, TMDS_RX2_SCL, TMDS_RX2_SDA, TMDS_TX1_0_N, TMDS_TX1_0_P, TMDS_TX1_1_N, TMDS_TX1_1_P, TMDS_TX1_2_N, TMDS_TX1_2_P, TMDS_TX1_CEC, TMDS_TX1_CLK_N, TMDS_TX1_CLK_P, TMDS_TX1_HOT, TMDS_TX1_SCL, TMDS_TX1_SDA, TMDS_TX2_0_N, TMDS_TX2_0_P, TMDS_TX2_1_N, TMDS_TX2_1_P, TMDS_TX2_2_N, TMDS_TX2_2_P, TMDS_TX2_CEC, TMDS_TX2_CLK_N, TMDS_TX2_CLK_P, TMDS_TX2_HOT, TMDS_TX2_SCL, TMDS_TX2_SDA
- wire segments 391 -> 522
Other:
- note removed: "LDO OUT FOR TX1"
- note removed: "LDO OUT FOR TX2"
